File: cherry/pcb/ganesha-cherry-left.kicad_pcb (KiCad board)
At the start: 2 copper layers, 275 x 124.6 mm, 210 parts, among them J1 MJ-4PP-9, J2 OLED, J3 MJ-4PP-9, J4 OLED, SW1 SW_PUSH, SW10 SW_PUSH, SW11 SW_PUSH, SW12 SW_PUSH, SW13 SW_PUSH, SW14 SW_PUSH, SW15 SW_PUSH, SW16 SW_PUSH, SW17 SW_PUSH, SW18 SW_PUSH, SW19 SW_PUSH, SW2 SW_PUSH, SW20 SW_PUSH, SW21 SW_PUSH, SW22 SW_PUSH, SW23 SW_PUSH, SW24 SW_PUSH, SW25 SW_PUSH, SW26 SW_PUSH, SW27 SW_PUSH, SW3 SW_PUSH, SW4 SW_PUSH, SW5 SW_PUSH, SW6 SW_PUSH, SW7 SW_PUSH, SW8 SW_PUSH, SW9 SW_PUSH, U1 ProMicro, U2 ProMicro

Commit message: minor revs and adding some design goals
Parts:
- removed D_R1, D_R10, D_R11, D_R12, D_R13, D_R14, D_R15, D_R16, D_R17, D_R18, D_R19, D_R2, D_R20, D_R21, D_R22, D_R23, D_R24, D_R25, D_R26, D_R27, D_R3, D_R4, D_R5, D_R6, D_R7, D_R8, D_R9: D, kbd:D3_SMD_v2
- removed J3: MJ-4PP-9, kbd:MJ-4PP-9_1side
- removed J4: OLED, kbd:OLED_1side
- removed LED_R_1, LED_R_10, LED_R_11, LED_R_12, LED_R_13, LED_R_14, LED_R_15, LED_R_16, LED_R_17, LED_R_18, LED_R_19, LED_R_2, LED_R_20, LED_R_21, LED_R_22, LED_R_23, LED_R_24, LED_R_25, LED_R_26, LED_R_27, LED_R_3, LED_R_4, LED_R_5, LED_R_6, LED_R_7, LED_R_8, LED_R_9: YS-SK6812MINI-E, kbd:YS-SK6812MINI-E
- removed LED_UR_1, LED_UR_2, LED_UR_3, LED_UR_4, LED_UR_5, LED_UR_6, LED_UR_7, LED_UR_8, LED_UR_9: WS2812B, LED_SMD:LED_WS2812B_PLCC4_5.0x5.0mm_P3.2mm
- removed REF** (x8): Breakaway_Tabs, kbd:Breakaway_Tabs
- removed RSW2: SW_PUSH, kbd:ResetSW_1side
- removed the Ref** at (168.9, 55.3)
- removed the Ref** at (269.2, 54.1)
- removed the Ref** at (191.1, 22.8)
- removed the Ref** at (267.1, 26.3)
- removed the Ref** at (224.0, 81.5)
- removed the Ref** at (154.4, 63.8)
- removed the Ref** at (177.4, 89.1)
- removed SW_R1, SW_R10, SW_R11, SW_R12, SW_R13, SW_R14, SW_R15, SW_R16, SW_R17, SW_R18, SW_R19, SW_R2, SW_R20, SW_R21, SW_R22, SW_R23, SW_R24, SW_R25, SW_R26, SW_R3, SW_R4, SW_R5, SW_R6, SW_R7, SW_R8, SW_R9: SW_PUSH, kbd:CherryMX_Hotswap
- removed SW_R27: SW_PUSH, kbd:CherryMX_Hotswap_1.5u
- removed U2: ProMicro, kbd:ProMicro_v3
Routing:
- net GND: track 1326.6 -> 849.6 mm, vias 28 -> 14
- net VDD: track 341.7 -> 0.00 mm, vias 2 -> 0
- net row2_r: track 252.3 -> 0.00 mm
- net VCC: track 920.2 -> 688.8 mm
- net row1_r: track 184.4 -> 0.00 mm, vias 2 -> 0
- net col0_r: track 175.8 -> 0.00 mm, vias 5 -> 0
- net row3_r: track 172.6 -> 0.00 mm, vias 2 -> 0
- net col1_r: track 150.7 -> 0.00 mm, vias 5 -> 0
- net GNDA: track 138.4 -> 0.00 mm, vias 1 -> 0
- net col3_r: track 133.0 -> 0.00 mm, vias 7 -> 0
- net col2_r: track 128.2 -> 0.00 mm, vias 5 -> 0
- net col4_r: track 115.5 -> 0.00 mm, vias 7 -> 0
- net row4_r: track 97.9 -> 0.00 mm, vias 2 -> 0
- net col5_r: track 86.8 -> 0.00 mm, vias 7 -> 0
- net Net-(LED_UR_7-Pad2): track 71.8 -> 0.00 mm, vias 2 -> 0
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Other:
- board size 275 x 124.6 mm -> 133.8 x 110.4 mm
- board text removed: "Corne Cherry v3.0.1 PCB Designed by foostan"
